Commit message: Fix WiFi connectivity, re-export meshes from STEP, update URDF
- Fix WiFi.config() ordering: must be called BEFORE WiFi.begin() to
  avoid EHOSTUNREACH errors on ESP32
- Re-export all STL meshes directly from STEP CAD with correct
  STEP→ROS axis mapping (X=-STEP_Y, Y=-STEP_X, Z=STEP_Z)
- Separate left/right wheel and bracket meshes for correct mirroring
- Add rear_mount mesh and caster (ball+housing merged)
- Update URDF with precise positions from STEP analysis
- Change wheel joint axis to Y and remove unnecessary rotations
- Add bracket and rear mount links to URDF
- Add joint_state_publisher to bringup launch for TF completeness
- Fix display.launch.py ParameterValue wrapping for Jazzy
- Fix odom publisher: zero velocities after 500ms cmd_vel timeout
- Add standalone ultrasonic proximity reading in WAITING_AGENT state
- Correct WHEEL_BASE to 81.4mm from STEP measurement

Co-Authored-By: Claude Opus 4.6 <noreply@anthropic.com>

File: ros2_ws/src/otto_description/urdf/otto_starter.urdf.xacro (robot description, xacro)
@@ -17,16 +17,23 @@
   <xacro:property name="variant" value="$(arg variant)"/>
   <!-- ============================== -->
-  <!-- Physical Properties             -->
+  <!-- Physical Properties (from STEP) -->
   <!-- ============================== -->
   <xacro:property name="wheel_radius" value="0.0245"/>
   <xacro:property name="wheel_width" value="0.0055"/>
-  <xacro:property name="wheel_base" value="0.108"/>
+  <xacro:property name="wheel_base" value="0.0814"/>
   <xacro:property name="body_width" value="0.075"/>
   <xacro:property name="body_depth" value="0.072"/>
-  <xacro:property name="body_height" value="0.062"/>
+  <xacro:property name="body_height" value="0.072"/>
   <xacro:property name="caster_radius" value="0.006"/>
-  <xacro:property name="head_width" value="0.052"/>
-  <xacro:property name="head_depth" value="0.052"/>
-  <xacro:property name="head_height" value="0.025"/>
+  <xacro:property name="head_width" value="0.062"/>
+  <xacro:property name="head_depth" value="0.016"/>
+  <xacro:property name="head_height" value="0.032"/>
+  <!-- Positions relative to base_link (at axle height, from STEP CAD) -->
+  <xacro:property name="body_offset_x" value="0.0231"/>  <!-- body center forward of axle -->
+  <xacro:property name="body_offset_z" value="0.0252"/>   <!-- body center above axle -->
+  <xacro:property name="face_offset_x" value="0.0607"/>   <!-- face forward of axle -->
+  <xacro:property name="face_offset_z" value="0.0262"/>   <!-- face above axle -->
+  <xacro:property name="caster_offset_x" value="0.0431"/> <!-- caster forward of axle -->
+  <xacro:property name="caster_offset_z" value="-0.0187"/><!-- caster below axle -->
   <!-- ============================== -->
   <!-- Material Definitions            -->
@@ -91,5 +98,5 @@
   <link name="base_link">
     <visual>
-      <origin xyz="0 0 0.016" rpy="0 0 0"/>
+      <origin xyz="${body_offset_x} 0 ${body_offset_z}" rpy="0 0 0"/>
       <geometry>
         <mesh filename="package://otto_description/meshes/body.stl"/>
@@ -98,5 +105,5 @@
     </visual>
     <collision>
-      <origin xyz="0 0 0.016" rpy="0 0 0"/>
+      <origin xyz="${body_offset_x} 0 ${body_offset_z}" rpy="0 0 0"/>
       <geometry>
         <box size="${body_depth} ${body_width} ${body_height}"/>
@@ -106,10 +113,10 @@
   </link>
   <!-- ============================== -->
-  <!-- Head Link (ultrasonic mount)    -->
+  <!-- Head Link (face plate at front) -->
   <!-- ============================== -->
   <joint name="head_joint" type="fixed">
     <parent link="base_link"/>
     <child link="head_link"/>
-    <origin xyz="0 0 ${body_height/2 + head_height/2 + 0.016}" rpy="0 0 0"/>
+    <origin xyz="${face_offset_x} 0 ${face_offset_z}" rpy="0 0 0"/>
   </joint>
   <link name="head_link">
@@ -163,5 +170,5 @@
     <parent link="base_link"/>
     <child link="led_ring_link"/>
-    <origin xyz="0.020 0 0.010" rpy="0 ${pi/2} 0"/>
+    <origin xyz="${body_offset_x} 0 ${body_offset_z + 0.030}" rpy="0 0 0"/>
   </joint>
   <link name="led_ring_link">
@@ -199,6 +206,6 @@
       <parent link="base_link"/>
       <child link="left_wheel_link"/>
-      <origin xyz="0 ${wheel_base/2} 0" rpy="${-pi/2} 0 0"/>
-      <axis xyz="0 0 1"/>
+      <origin xyz="0 ${wheel_base/2} 0" rpy="0 0 0"/>
+      <axis xyz="0 1 0"/>
       <dynamics damping="0.01" friction="0.01"/>
     </joint>
@@ -206,9 +213,10 @@
       <visual>
         <geometry>
-          <mesh filename="package://otto_description/meshes/wheel.stl"/>
+          <mesh filename="package://otto_description/meshes/wheel_left.stl"/>
         </geometry>
         <material name="rubber_black"/>
       </visual>
       <collision>
+        <origin xyz="0 0 0" rpy="${pi/2} 0 0"/>
         <geometry>
           <cylinder radius="${wheel_radius}" length="${wheel_width}"/>
@@ -217,10 +225,28 @@
       <xacro:cylinder_inertia m="0.015" r="${wheel_radius}" h="${wheel_width}"/>
     </link>
+    <!-- Left Bracket -->
+    <joint name="left_bracket_joint" type="fixed">
+      <parent link="base_link"/>
+      <child link="left_bracket_link"/>
+      <origin xyz="0 ${wheel_base/2} 0" rpy="0 0 0"/>
+    </joint>
+    <link name="left_bracket_link">
+      <visual>
+        <geometry>
+          <mesh filename="package://otto_description/meshes/bracket_left.stl"/>
+        </geometry>
+        <material name="otto_white"/>
+      </visual>
+      <inertial>
+        <mass value="0.005"/>
+        <inertia ixx="1e-7" ixy="0" ixz="0" iyy="1e-7" iyz="0" izz="1e-7"/>
+      </inertial>
+    </link>
     <!-- Right Wheel -->
     <joint name="right_wheel_joint" type="continuous">
       <parent link="base_link"/>
       <child link="right_wheel_link"/>
-      <origin xyz="0 ${-wheel_base/2} 0" rpy="${-pi/2} 0 0"/>
-      <axis xyz="0 0 1"/>
+      <origin xyz="0 ${-wheel_base/2} 0" rpy="0 0 0"/>
+      <axis xyz="0 1 0"/>
       <dynamics damping="0.01" friction="0.01"/>
     </joint>
@@ -228,9 +254,10 @@
       <visual>
         <geometry>
-          <mesh filename="package://otto_description/meshes/wheel.stl"/>
+          <mesh filename="package://otto_description/meshes/wheel_right.stl"/>
         </geometry>
         <material name="rubber_black"/>
       </visual>
       <collision>
+        <origin xyz="0 0 0" rpy="${pi/2} 0 0"/>
         <geometry>
           <cylinder radius="${wheel_radius}" length="${wheel_width}"/>
@@ -239,9 +266,28 @@
       <xacro:cylinder_inertia m="0.015" r="${wheel_radius}" h="${wheel_width}"/>
     </link>
-    <!-- Ball Caster (rear support) -->
+    <!-- Right Bracket -->
+    <joint name="right_bracket_joint" type="fixed">
+      <parent link="base_link"/>
+      <child link="right_bracket_link"/>
+      <origin xyz="0 ${-wheel_base/2} 0" rpy="0 0 0"/>
+    </joint>
+    <link name="right_bracket_link">
+      <visual>
+        <origin xyz="0 0 0" rpy="0 0 0"/>
+        <geometry>
+          <mesh filename="package://otto_description/meshes/bracket_right.stl"/>
+        </geometry>
+        <material name="otto_white"/>
+      </visual>
+      <inertial>
+        <mass value="0.005"/>
+        <inertia ixx="1e-7" ixy="0" ixz="0" iyy="1e-7" iyz="0" izz="1e-7"/>
+      </inertial>
+    </link>
+    <!-- Ball Caster (front support) -->
     <joint name="caster_joint" type="fixed">
       <parent link="base_link"/>
       <child link="caster_link"/>
-      <origin xyz="-0.030 0 ${-wheel_radius + caster_radius}" rpy="0 0 0"/>
+      <origin xyz="${caster_offset_x} 0 ${caster_offset_z}" rpy="0 0 0"/>
     </joint>
     <link name="caster_link">
@@ -258,4 +304,22 @@
       </collision>
       <xacro:sphere_inertia m="0.007" r="${caster_radius}"/>
+    </link>
+    <!-- Rear Mount -->
+    <joint name="rear_mount_joint" type="fixed">
+      <parent link="base_link"/>
+      <child link="rear_mount_link"/>
+      <origin xyz="0.003 0 0" rpy="0 0 0"/>
+    </joint>
+    <link name="rear_mount_link">
+      <visual>
+        <geometry>
+          <mesh filename="package://otto_description/meshes/rear_mount.stl"/>
+        </geometry>
+        <material name="otto_white"/>
+      </visual>
+      <inertial>
+        <mass value="0.005"/>
+        <inertia ixx="1e-7" ixy="0" ixz="0" iyy="1e-7" iyz="0" izz="1e-7"/>
+      </inertial>
     </link>
     <!-- IR Line Sensors (bottom, pointing down) -->

Commit message: Update meshes from new ZGX Otto STEP design
- Move hardware/ZGX Otto.step from project root (gitignored as large binary)
- Rewrite scripts/export_meshes.py: named-part classification for new STEP
  structure (Top/Middle/Bottom/Logo → body, Lines→face, Wheels, Ballcaster,
  Battery Cover); prints URDF origin for new parts
- Regenerate all STL meshes from new design (body, face, wheel_left,
  wheel_right, caster, battery_cover)
- URDF: remove bracket_left/right and rear_mount links (not in new design);
  add battery_cover_link with origin from bounding box export
- Add docs/hardware.md: CAD source location, re-export instructions,
  coordinate transform reference
- Add hardware/ to .gitignore and README project structure

Co-Authored-By: Claude Sonnet 4.6 <noreply@anthropic.com>

File: ros2_ws/src/otto_description/urdf/otto_starter.urdf.xacro (robot description, xacro)
@@ -225,22 +225,4 @@
       <xacro:cylinder_inertia m="0.015" r="${wheel_radius}" h="${wheel_width}"/>
     </link>
-    <!-- Left Bracket -->
-    <joint name="left_bracket_joint" type="fixed">
-      <parent link="base_link"/>
-      <child link="left_bracket_link"/>
-      <origin xyz="0 ${wheel_base/2} 0" rpy="0 0 0"/>
-    </joint>
-    <link name="left_bracket_link">
-      <visual>
-        <geometry>
-          <mesh filename="package://otto_description/meshes/bracket_left.stl"/>
-        </geometry>
-        <material name="otto_white"/>
-      </visual>
-      <inertial>
-        <mass value="0.005"/>
-        <inertia ixx="1e-7" ixy="0" ixz="0" iyy="1e-7" iyz="0" izz="1e-7"/>
-      </inertial>
-    </link>
     <!-- Right Wheel -->
     <joint name="right_wheel_joint" type="continuous">
@@ -266,23 +248,4 @@
       <xacro:cylinder_inertia m="0.015" r="${wheel_radius}" h="${wheel_width}"/>
     </link>
-    <!-- Right Bracket -->
-    <joint name="right_bracket_joint" type="fixed">
-      <parent link="base_link"/>
-      <child link="right_bracket_link"/>
-      <origin xyz="0 ${-wheel_base/2} 0" rpy="0 0 0"/>
-    </joint>
-    <link name="right_bracket_link">
-      <visual>
-        <origin xyz="0 0 0" rpy="0 0 0"/>
-        <geometry>
-          <mesh filename="package://otto_description/meshes/bracket_right.stl"/>
-        </geometry>
-        <material name="otto_white"/>
-      </visual>
-      <inertial>
-        <mass value="0.005"/>
-        <inertia ixx="1e-7" ixy="0" ixz="0" iyy="1e-7" iyz="0" izz="1e-7"/>
-      </inertial>
-    </link>
     <!-- Ball Caster (front support) -->
     <joint name="caster_joint" type="fixed">
@@ -305,20 +268,20 @@
       <xacro:sphere_inertia m="0.007" r="${caster_radius}"/>
     </link>
-    <!-- Rear Mount -->
-    <joint name="rear_mount_joint" type="fixed">
-      <parent link="base_link"/>
-      <child link="rear_mount_link"/>
-      <origin xyz="0.003 0 0" rpy="0 0 0"/>
-    </joint>
-    <link name="rear_mount_link">
-      <visual>
-        <geometry>
-          <mesh filename="package://otto_description/meshes/rear_mount.stl"/>
+    <!-- Battery Cover (rear panel, includes HP logo) -->
+    <joint name="battery_cover_joint" type="fixed">
+      <parent link="base_link"/>
+      <child link="battery_cover_link"/>
+      <origin xyz="-0.0065 0 0.0197" rpy="0 0 0"/>
+    </joint>
+    <link name="battery_cover_link">
+      <visual>
+        <geometry>
+          <mesh filename="package://otto_description/meshes/battery_cover.stl"/>
         </geometry>
         <material name="otto_white"/>
       </visual>
       <inertial>
-        <mass value="0.005"/>
-        <inertia ixx="1e-7" ixy="0" ixz="0" iyy="1e-7" iyz="0" izz="1e-7"/>
+        <mass value="0.010"/>
+        <inertia ixx="1e-6" ixy="0" ixz="0" iyy="1e-6" iyz="0" izz="1e-6"/>
       </inertial>
     </link>

Commit message: Fix URDF mesh positioning: proper STEP→ROS coordinate transform
- export_meshes.py: replace scale_stl with transform_stl that applies the
  full STEP→ROS axis remap (STEP -Y→ROS +X, STEP -X→ROS +Y) and centers
  each mesh at its bounding-box centroid so all visual origins are (0,0,0)
- Add STEP_AXLE_Y=23mm so joint origins are relative to the wheel axle
  center (base_link) rather than the arbitrary STEP file origin
- Update all URDF joint/visual origins from re-exported centroid values:
  wheel_base 81.4→83.4mm, body/face/caster/battery_cover positions corrected
- Regenerate all STL meshes in ROS coordinate space

Co-Authored-By: Claude Sonnet 4.6 <noreply@anthropic.com>

File: ros2_ws/src/otto_description/urdf/otto_starter.urdf.xacro (robot description, xacro)
@@ -21,5 +21,5 @@
   <xacro:property name="wheel_radius" value="0.0245"/>
   <xacro:property name="wheel_width" value="0.0055"/>
-  <xacro:property name="wheel_base" value="0.0814"/>
+  <xacro:property name="wheel_base" value="0.0834"/>  <!-- 2 × 41.7 mm from STEP -->
   <xacro:property name="body_width" value="0.075"/>
   <xacro:property name="body_depth" value="0.072"/>
@@ -29,11 +29,11 @@
   <xacro:property name="head_depth" value="0.016"/>
   <xacro:property name="head_height" value="0.032"/>
-  <!-- Positions relative to base_link (at axle height, from STEP CAD) -->
-  <xacro:property name="body_offset_x" value="0.0231"/>  <!-- body center forward of axle -->
-  <xacro:property name="body_offset_z" value="0.0252"/>   <!-- body center above axle -->
-  <xacro:property name="face_offset_x" value="0.0607"/>   <!-- face forward of axle -->
-  <xacro:property name="face_offset_z" value="0.0262"/>   <!-- face above axle -->
-  <xacro:property name="caster_offset_x" value="0.0431"/> <!-- caster forward of axle -->
-  <xacro:property name="caster_offset_z" value="-0.0187"/><!-- caster below axle -->
+  <!-- Positions relative to base_link (at axle centre, from export_meshes.py output) -->
+  <xacro:property name="body_offset_x" value="0.0230"/>   <!-- body centroid forward of axle -->
+  <xacro:property name="body_offset_z" value="0.0220"/>   <!-- body centroid above axle -->
+  <xacro:property name="face_offset_x" value="0.0605"/>   <!-- face centroid forward of axle -->
+  <xacro:property name="face_offset_z" value="0.0260"/>   <!-- face centroid above axle -->
+  <xacro:property name="caster_offset_x" value="0.0430"/> <!-- caster centroid forward of axle -->
+  <xacro:property name="caster_offset_z" value="-0.0190"/><!-- caster centroid below axle -->
   <!-- ============================== -->
   <!-- Material Definitions            -->
@@ -99,4 +99,5 @@
     <visual>
       <origin xyz="${body_offset_x} 0 ${body_offset_z}" rpy="0 0 0"/>
+      <!-- mesh is centered at its own centroid; this origin places it in base_link -->
       <geometry>
         <mesh filename="package://otto_description/meshes/body.stl"/>
@@ -272,5 +273,5 @@
       <parent link="base_link"/>
       <child link="battery_cover_link"/>
-      <origin xyz="-0.0065 0 0.0197" rpy="0 0 0"/>
+      <origin xyz="0.0165 0 0.0197" rpy="0 0 0"/>
     </joint>
     <link name="battery_cover_link">
