Commit message: Rebuild URDF and meshes from updated 24MB STEP file
- Rewrite export_meshes.py: auto-computes AXLE_Z/AXLE_Y from wheel
  geometry, bounding-box classification, STEP→ROS coordinate transform
  applied at vertex level so visual origins are all (0 0 0)
- Export 8 STL meshes: body, wheel_left/right, caster, led_ring,
  ultrasonic, line_sensor_left/right
- Remove old meshes: battery_cover, bracket_left/right, face, rear_mount
- Rewrite otto_starter.urdf.xacro: base_footprint→base_link link tree,
  continuous wheel joints on Y axis, 15 LED child frames, all joint
  origins from export script output
- Add otto_visualizer.py: MarkerArray for LED ring, colour sphere for
  sonar distance; wired into otto_microros.launch.py
- Add otto.rviz: RobotModel, TF, MarkerArray, Marker, Range displays
- Update CMakeLists.txt to install otto_visualizer.py
- Add visualization_msgs exec_depend to package.xml

Co-Authored-By: Claude Sonnet 4.6 <noreply@anthropic.com>

File: ros2_ws/src/otto_description/urdf/otto_starter.urdf.xacro (robot description, xacro)
@@ -1,69 +1,56 @@
-<?xml version="1.0" encoding="UTF-8"?>
+<?xml version="1.0"?>
 <!--
-  HP Robots Otto Starter - Parameterized URDF (Xacro)
-  ====================================================
-  Supports both wheeled (Starter Kit) and biped variants via xacro arg.
-  Usage:
-    Wheeled: xacro otto_starter.urdf.xacro variant:=wheeled
-    Biped:   xacro otto_starter.urdf.xacro variant:=biped
-  Coordinate frame: X forward, Y left, Z up (REP-103)
-  Units: meters, radians, kg
+  Otto Starter Kit — URDF (xacro)
+  Coordinate system: ROS REP-103 (X=forward, Y=left, Z=up)
+  base_footprint : ground plane (Z = 0)
+  base_link      : wheel axle height (Z = wheel_radius above ground)
+  Mesh joint origins are printed by scripts/export_meshes.py — update here
+  if the STEP file is re-exported.
+  All STL meshes are pre-centred at their joint origin so visual/collision
+  origins are (0 0 0) throughout.
 -->
 <robot name="otto_starter" xmlns:xacro="http://www.ros.org/wiki/xacro">
-  <!-- ============================== -->
-  <!-- Arguments                       -->
-  <!-- ============================== -->
-  <xacro:arg name="variant" default="wheeled"/>
-  <xacro:property name="variant" value="$(arg variant)"/>
-  <!-- ============================== -->
-  <!-- Physical Properties (from STEP) -->
-  <!-- ============================== -->
-  <xacro:property name="wheel_radius" value="0.0245"/>
-  <xacro:property name="wheel_width" value="0.0055"/>
-  <xacro:property name="wheel_base" value="0.0834"/>  <!-- 2 × 41.7 mm from STEP -->
-  <xacro:property name="body_width" value="0.075"/>
-  <xacro:property name="body_depth" value="0.072"/>
-  <xacro:property name="body_height" value="0.072"/>
-  <xacro:property name="caster_radius" value="0.006"/>
-  <xacro:property name="head_width" value="0.062"/>
-  <xacro:property name="head_depth" value="0.016"/>
-  <xacro:property name="head_height" value="0.032"/>
-  <!-- Positions relative to base_link (at axle centre, from export_meshes.py output) -->
-  <xacro:property name="body_offset_x" value="0.0230"/>   <!-- body centroid forward of axle -->
-  <xacro:property name="body_offset_z" value="0.0220"/>   <!-- body centroid above axle -->
-  <xacro:property name="face_offset_x" value="0.0605"/>   <!-- face centroid forward of axle -->
-  <xacro:property name="face_offset_z" value="0.0260"/>   <!-- face centroid above axle -->
-  <xacro:property name="caster_offset_x" value="0.0430"/> <!-- caster centroid forward of axle -->
-  <xacro:property name="caster_offset_z" value="-0.0190"/><!-- caster centroid below axle -->
-  <!-- ============================== -->
-  <!-- Material Definitions            -->
-  <!-- ============================== -->
+  <!-- ══════════════════════════════════════════════════════════════════ -->
+  <!--  Parameters                                                        -->
+  <!-- ══════════════════════════════════════════════════════════════════ -->
+  <xacro:property name="wheel_radius"   value="0.0245"/>   <!-- m -->
+  <xacro:property name="wheel_base"     value="0.0913"/>   <!-- m  (track width) -->
+  <xacro:property name="wheel_width"    value="0.008"/>    <!-- m -->
+  <xacro:property name="wheel_mass"     value="0.020"/>    <!-- kg -->
+  <xacro:property name="body_mass"      value="0.300"/>    <!-- kg -->
+  <xacro:property name="caster_mass"    value="0.010"/>    <!-- kg -->
+  <!-- ══════════════════════════════════════════════════════════════════ -->
+  <!--  Materials                                                         -->
+  <!-- ══════════════════════════════════════════════════════════════════ -->
   <material name="otto_white">
     <color rgba="0.95 0.95 0.95 1.0"/>
   </material>
   <material name="otto_blue">
-    <color rgba="0.2 0.4 0.8 1.0"/>
+    <color rgba="0.12 0.47 0.71 1.0"/>
   </material>
   <material name="otto_dark">
     <color rgba="0.15 0.15 0.15 1.0"/>
   </material>
-  <material name="otto_orange">
-    <color rgba="1.0 0.5 0.0 1.0"/>
+  <material name="rubber_black">
+    <color rgba="0.08 0.08 0.08 1.0"/>
+  </material>
+  <material name="led_white">
+    <color rgba="1.0 1.0 1.0 1.0"/>
   </material>
   <material name="sensor_green">
     <color rgba="0.0 0.8 0.2 0.8"/>
   </material>
-  <material name="rubber_black">
-    <color rgba="0.1 0.1 0.1 1.0"/>
-  </material>
-  <!-- ============================== -->
-  <!-- Inertia Macros                  -->
-  <!-- ============================== -->
-  <xacro:macro name="box_inertia" params="m w d h">
+  <material name="pcb_green">
+    <color rgba="0.05 0.35 0.05 1.0"/>
+  </material>
+  <!-- ══════════════════════════════════════════════════════════════════ -->
+  <!--  Helper macro: simple box inertia                                  -->
+  <!-- ══════════════════════════════════════════════════════════════════ -->
+  <xacro:macro name="box_inertia" params="m x y z">
     <inertial>
       <mass value="${m}"/>
-      <inertia ixx="${m*(d*d+h*h)/12}" ixy="0" ixz="0"
-               iyy="${m*(w*w+h*h)/12}" iyz="0"
-               izz="${m*(w*w+d*d)/12}"/>
+      <inertia ixx="${m*(y*y+z*z)/12}" ixy="0" ixz="0"
+               iyy="${m*(x*x+z*z)/12}" iyz="0"
+               izz="${m*(x*x+y*y)/12}"/>
     </inertial>
   </xacro:macro>
@@ -76,28 +63,27 @@
     </inertial>
   </xacro:macro>
-  <xacro:macro name="sphere_inertia" params="m r">
-    <inertial>
-      <mass value="${m}"/>
-      <inertia ixx="${2*m*r*r/5}" ixy="0" ixz="0"
-               iyy="${2*m*r*r/5}" iyz="0"
-               izz="${2*m*r*r/5}"/>
-    </inertial>
-  </xacro:macro>
-  <!-- ============================== -->
-  <!-- Base Footprint (ground plane)   -->
-  <!-- ============================== -->
+  <!-- ══════════════════════════════════════════════════════════════════ -->
+  <!--  base_footprint — ground reference frame (Z = 0)                  -->
+  <!-- ══════════════════════════════════════════════════════════════════ -->
   <link name="base_footprint"/>
   <joint name="base_footprint_joint" type="fixed">
     <parent link="base_footprint"/>
-    <child link="base_link"/>
+    <child  link="base_link"/>
     <origin xyz="0 0 ${wheel_radius}" rpy="0 0 0"/>
   </joint>
-  <!-- ============================== -->
-  <!-- Base Link (body center at axle) -->
-  <!-- ============================== -->
+  <!-- ══════════════════════════════════════════════════════════════════ -->
+  <!--  base_link — wheel axle height                                     -->
+  <!-- ══════════════════════════════════════════════════════════════════ -->
   <link name="base_link">
-    <visual>
-      <origin xyz="${body_offset_x} 0 ${body_offset_z}" rpy="0 0 0"/>
-      <!-- mesh is centered at its own centroid; this origin places it in base_link -->
+    <xacro:box_inertia m="${body_mass}" x="0.072" y="0.072" z="0.072"/>
+  </link>
+  <!-- ══════════════════════════════════════════════════════════════════ -->
+  <!--  Body shell                                                        -->
+  <!--  joint xyz from export_meshes.py:                                 -->
+  <!--    body: joint xyz="0.0231 0.0000 0.0220"                         -->
+  <!-- ══════════════════════════════════════════════════════════════════ -->
+  <link name="body_link">
+    <visual>
+      <origin xyz="0 0 0" rpy="0 0 0"/>
       <geometry>
         <mesh filename="package://otto_description/meshes/body.stl"/>
@@ -106,419 +92,215 @@
     </visual>
     <collision>
-      <origin xyz="${body_offset_x} 0 ${body_offset_z}" rpy="0 0 0"/>
-      <geometry>
-        <box size="${body_depth} ${body_width} ${body_height}"/>
-      </geometry>
-    </collision>
-    <xacro:box_inertia m="0.120" w="${body_width}" d="${body_depth}" h="${body_height}"/>
-  </link>
-  <!-- ============================== -->
-  <!-- Head Link (face plate at front) -->
-  <!-- ============================== -->
-  <joint name="head_joint" type="fixed">
-    <parent link="base_link"/>
-    <child link="head_link"/>
-    <origin xyz="${face_offset_x} 0 ${face_offset_z}" rpy="0 0 0"/>
-  </joint>
-  <link name="head_link">
-    <visual>
-      <origin xyz="0 0 0" rpy="0 0 0"/>
-      <geometry>
-        <mesh filename="package://otto_description/meshes/face.stl"/>
-      </geometry>
-      <material name="otto_blue"/>
-    </visual>
-    <collision>
-      <origin xyz="0 0 0" rpy="0 0 0"/>
-      <geometry>
-        <box size="${head_depth} ${head_width} ${head_height}"/>
-      </geometry>
-    </collision>
-    <xacro:box_inertia m="0.025" w="${head_width}" d="${head_depth}" h="${head_height}"/>
-  </link>
-  <!-- ============================== -->
-  <!-- Ultrasonic Sensor Frame         -->
-  <!-- ============================== -->
+      <origin xyz="0 0 0" rpy="0 0 0"/>
+      <geometry>
+        <box size="0.072 0.072 0.072"/>
+      </geometry>
+    </collision>
+    <xacro:box_inertia m="${body_mass}" x="0.072" y="0.072" z="0.072"/>
+  </link>
+  <joint name="body_joint" type="fixed">
+    <parent link="base_link"/>
+    <child  link="body_link"/>
+    <origin xyz="0.0231 0.0000 0.0220" rpy="0 0 0"/>
+  </joint>
+  <!-- ══════════════════════════════════════════════════════════════════ -->
+  <!--  Wheels                                                            -->
+  <!--  joint xyz from export_meshes.py:                                 -->
+  <!--    wheel_left:  joint xyz="-0.0000 0.0416 0.0000"                 -->
+  <!--    wheel_right: joint xyz="-0.0000 -0.0416 0.0000"                -->
+  <!--  Meshes centred at axle midpoint — rotate around Y correctly.     -->
+  <!-- ══════════════════════════════════════════════════════════════════ -->
+  <link name="left_wheel_link">
+    <visual>
+      <origin xyz="0 0 0" rpy="0 0 0"/>
+      <geometry>
+        <mesh filename="package://otto_description/meshes/wheel_left.stl"/>
+      </geometry>
+      <material name="rubber_black"/>
+    </visual>
+    <collision>
+      <origin xyz="0 0 0" rpy="${pi/2} 0 0"/>
+      <geometry>
+        <cylinder radius="${wheel_radius}" length="${wheel_width}"/>
+      </geometry>
+    </collision>
+    <xacro:cylinder_inertia m="${wheel_mass}" r="${wheel_radius}" h="${wheel_width}"/>
+  </link>
+  <joint name="left_wheel_joint" type="continuous">
+    <parent link="base_link"/>
+    <child  link="left_wheel_link"/>
+    <origin xyz="-0.0000 0.0416 0.0000" rpy="0 0 0"/>
+    <axis xyz="0 1 0"/>
+  </joint>
+  <link name="right_wheel_link">
+    <visual>
+      <origin xyz="0 0 0" rpy="0 0 0"/>
+      <geometry>
+        <mesh filename="package://otto_description/meshes/wheel_right.stl"/>
+      </geometry>
+      <material name="rubber_black"/>
+    </visual>
+    <collision>
+      <origin xyz="0 0 0" rpy="${pi/2} 0 0"/>
+      <geometry>
+        <cylinder radius="${wheel_radius}" length="${wheel_width}"/>
+      </geometry>
+    </collision>
+    <xacro:cylinder_inertia m="${wheel_mass}" r="${wheel_radius}" h="${wheel_width}"/>
+  </link>
+  <joint name="right_wheel_joint" type="continuous">
+    <parent link="base_link"/>
+    <child  link="right_wheel_link"/>
+    <origin xyz="-0.0000 -0.0416 0.0000" rpy="0 0 0"/>
+    <axis xyz="0 1 0"/>
+  </joint>
+  <!-- ══════════════════════════════════════════════════════════════════ -->
+  <!--  Caster (front ball caster)                                        -->
+  <!-- ══════════════════════════════════════════════════════════════════ -->
+  <link name="caster_link">
+    <visual>
+      <origin xyz="0 0 0" rpy="0 0 0"/>
+      <geometry>
+        <mesh filename="package://otto_description/meshes/caster.stl"/>
+      </geometry>
+      <material name="otto_dark"/>
+    </visual>
+    <collision>
+      <origin xyz="0 0 0" rpy="0 0 0"/>
+      <geometry>
+        <sphere radius="0.006"/>
+      </geometry>
+    </collision>
+    <xacro:box_inertia m="${caster_mass}" x="0.012" y="0.012" z="0.012"/>
+  </link>
+  <joint name="caster_joint" type="fixed">
+    <parent link="base_link"/>
+    <child  link="caster_link"/>
+    <origin xyz="0.0430 0.0000 -0.0190" rpy="0 0 0"/>
+  </joint>
+  <!-- ══════════════════════════════════════════════════════════════════ -->
+  <!--  LED Ring                                                          -->
+  <!--  joint xyz from export_meshes.py:                                 -->
+  <!--    led_ring: joint xyz="0.0231 0.0001 0.0516"                     -->
+  <!-- ══════════════════════════════════════════════════════════════════ -->
+  <link name="led_ring_link">
+    <visual>
+      <origin xyz="0 0 0" rpy="0 0 0"/>
+      <geometry>
+        <mesh filename="package://otto_description/meshes/led_ring.stl"/>
+      </geometry>
+      <material name="pcb_green"/>
+    </visual>
+    <collision>
+      <origin xyz="0 0 0" rpy="0 0 0"/>
+      <geometry>
+        <cylinder radius="0.025" length="0.002"/>
+      </geometry>
+    </collision>
+    <xacro:box_inertia m="0.005" x="0.05" y="0.05" z="0.002"/>
+  </link>
+  <joint name="led_ring_joint" type="fixed">
+    <parent link="base_link"/>
+    <child  link="led_ring_link"/>
+    <origin xyz="0.0231 0.0001 0.0516" rpy="0 0 0"/>
+  </joint>
+  <!-- ── Individual LED frames (positions relative to base_link) ──────
+       Values from export_meshes.py LED ring frame positions output.
+       These are used by otto_visualizer to publish marker poses.       -->
+  <xacro:macro name="led_frame" params="n x y z">
+    <link name="led_${n}_link"/>
+    <joint name="led_${n}_joint" type="fixed">
+      <parent link="base_link"/>
+      <child  link="led_${n}_link"/>
+      <origin xyz="${x} ${y} ${z}" rpy="0 0 0"/>
+    </joint>
+  </xacro:macro>
+  <xacro:led_frame n="0"  x="0.0049" y="-0.0104" z="0.0532"/>
+  <xacro:led_frame n="1"  x="0.0126" y="-0.0181" z="0.0532"/>
+  <xacro:led_frame n="2"  x="0.0231" y="-0.0209" z="0.0532"/>
+  <xacro:led_frame n="3"  x="0.0336" y="-0.0181" z="0.0532"/>
+  <xacro:led_frame n="4"  x="0.0412" y="-0.0104" z="0.0532"/>
+  <xacro:led_frame n="5"  x="0.0536" y="-0.0130" z="0.0310"/>
+  <xacro:led_frame n="6"  x="0.0441" y=" 0.0001" z="0.0532"/>
+  <xacro:led_frame n="7"  x="0.0231" y=" 0.0001" z="0.0532"/>
+  <xacro:led_frame n="8"  x="0.0021" y=" 0.0001" z="0.0532"/>
+  <xacro:led_frame n="9"  x="0.0536" y=" 0.0130" z="0.0310"/>
+  <xacro:led_frame n="10" x="0.0412" y=" 0.0106" z="0.0532"/>
+  <xacro:led_frame n="11" x="0.0336" y=" 0.0183" z="0.0532"/>
+  <xacro:led_frame n="12" x="0.0231" y=" 0.0211" z="0.0532"/>
+  <xacro:led_frame n="13" x="0.0126" y=" 0.0183" z="0.0532"/>
+  <xacro:led_frame n="14" x="0.0049" y=" 0.0106" z="0.0532"/>
+  <!-- ══════════════════════════════════════════════════════════════════ -->
+  <!--  Ultrasonic sensor                                                 -->
+  <!-- ══════════════════════════════════════════════════════════════════ -->
+  <link name="ultrasonic_link">
+    <visual>
+      <origin xyz="0 0 0" rpy="0 0 0"/>
+      <geometry>
+        <mesh filename="package://otto_description/meshes/ultrasonic.stl"/>
+      </geometry>
+      <material name="sensor_green"/>
+    </visual>
+    <collision>
+      <origin xyz="0 0 0" rpy="0 0 0"/>
+      <geometry>
+        <box size="0.010 0.005 0.006"/>
+      </geometry>
+    </collision>
+    <xacro:box_inertia m="0.002" x="0.010" y="0.005" z="0.006"/>
+  </link>
   <joint name="ultrasonic_joint" type="fixed">
-    <parent link="head_link"/>
-    <child link="ultrasonic_link"/>
-    <origin xyz="0.026 0 0" rpy="0 0 0"/>
-  </joint>
-  <link name="ultrasonic_link">
-    <visual>
-      <origin xyz="0.003 0.008 0" rpy="0 ${pi/2} 0"/>
-      <geometry>
-        <cylinder radius="0.008" length="0.006"/>
-      </geometry>
-      <material name="sensor_green"/>
-    </visual>
-    <visual>
-      <origin xyz="0.003 -0.008 0" rpy="0 ${pi/2} 0"/>
-      <geometry>
-        <cylinder radius="0.008" length="0.006"/>
-      </geometry>
-      <material name="sensor_green"/>
-    </visual>
-    <inertial>
-      <mass value="0.005"/>
-      <inertia ixx="1e-7" ixy="0" ixz="0" iyy="1e-7" iyz="0" izz="1e-7"/>
-    </inertial>
-  </link>
-  <!-- ============================== -->
-  <!-- LED Ring (visual only)          -->
-  <!-- ============================== -->
-  <joint name="led_ring_joint" type="fixed">
-    <parent link="base_link"/>
-    <child link="led_ring_link"/>
-    <origin xyz="${body_offset_x} 0 ${body_offset_z + 0.030}" rpy="0 0 0"/>
-  </joint>
-  <link name="led_ring_link">
-    <visual>
-      <geometry>
-        <cylinder radius="0.018" length="0.003"/>
-      </geometry>
-      <material name="otto_orange"/>
-    </visual>
-    <inertial>
-      <mass value="0.003"/>
-      <inertia ixx="1e-7" ixy="0" ixz="0" iyy="1e-7" iyz="0" izz="1e-7"/>
-    </inertial>
-  </link>
-  <!-- ============================== -->
-  <!-- IMU Link (placeholder)          -->
-  <!-- ============================== -->
+    <parent link="base_link"/>
+    <child  link="ultrasonic_link"/>
+    <origin xyz="0.0465 -0.0000 0.0049" rpy="0 0 0"/>
+  </joint>
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
Commit message: Fix mesh classification and raise tessellation quality
Classification fixes:
- Body: add front face panel condition (w>55, h>25, thin, front-centre)
  so the 66x11x36mm face plate is no longer skipped
- Ultrasonic: add abs(cx)<5 guard to exclude servo motors at cx=±13mm
  that were wrongly matching the sensor housing condition

Tessellation quality (tolerance=0.05mm, angular=0.02rad):
- 10x finer than previous settings — fillets and curved surfaces now
  properly represented; file size increases are intentional

URDF joint origin updates from re-export:
- body: 0.0231 → 0.0265 (centroid shifted with face plate included)
- ultrasonic: 0.0465/0.0049 → 0.0509/0.0200 (corrected to housing only)

Co-Authored-By: Claude Sonnet 4.6 <noreply@anthropic.com>

File: ros2_ws/src/otto_description/urdf/otto_starter.urdf.xacro (robot description, xacro)
@@ -102,5 +102,5 @@
     <parent link="base_link"/>
     <child  link="body_link"/>
-    <origin xyz="0.0231 0.0000 0.0220" rpy="0 0 0"/>
+    <origin xyz="0.0265 -0.0000 0.0220" rpy="0 0 0"/>
   </joint>
   <!-- ══════════════════════════════════════════════════════════════════ -->
@@ -181,6 +181,5 @@
   <!-- ══════════════════════════════════════════════════════════════════ -->
   <!--  LED Ring                                                          -->
-  <!--  joint xyz from export_meshes.py:                                 -->
-  <!--    led_ring: joint xyz="0.0231 0.0001 0.0516"                     -->
+  <!--  joint xyz from export_meshes.py output                           -->
   <!-- ══════════════════════════════════════════════════════════════════ -->
   <link name="led_ring_link">
@@ -253,5 +252,5 @@
     <parent link="base_link"/>
     <child  link="ultrasonic_link"/>
-    <origin xyz="0.0465 -0.0000 0.0049" rpy="0 0 0"/>
+    <origin xyz="0.0509 0.0000 0.0200" rpy="0 0 0"/>
   </joint>
   <!-- Sensor ray origin — midpoint between transducers, pointing forward -->
