Commit message: Split body/wheel meshes by named STEP groups; fix geometry mirror
- export_meshes.py: rewrite using OCP CAF names for exact part grouping
  - Body: 6 sub-meshes (shell, clips, top, logo lines, bottom, face panel)
  - Wheels: 4 sub-meshes split by diameter (tire ≈49mm vs rim ≤45mm)
  - Fix det=-1 geometry mirror: change ros_y = +step_x (det=+1 proper
    rotation), update normals to (-ny, nx, nz), remove winding swap
  - Line sensor names no longer swapped (STEP Left/Right match physical)
  - Wheel tire threshold: dia > 46mm (was > 50mm, outer tire is 49mm)
  - body_bottom/face: geometric search across all CAF-named solids

- urdf/otto_starter.urdf.xacro:
  - Multiple <visual> elements per body and wheel links for colouring:
    shell/clips/face → dark_grey; top dome → white; logos/bottom → black
    wheel rim → dark_grey; wheel tire → rubber_black
  - New materials: otto_dark_grey, otto_black
  - Updated joint origins from new export (body, ultrasonic, line sensors)
  - 13 LED frames (was 15); correct LED pad positions from CAF 'LED Ring'
  - wheel_base 0.0913→0.0833m (axle-to-axle, not bounding-box width)

- otto_visualizer.py: NUM_LEDS 15→13

Co-Authored-By: Claude Sonnet 4.6 <noreply@anthropic.com>

File: ros2_ws/src/otto_description/urdf/otto_starter.urdf.xacro (robot description, xacro)
@@ -7,6 +7,8 @@
   Mesh joint origins are printed by scripts/export_meshes.py — update here
   if the STEP file is re-exported.
-  All STL meshes are pre-centred at their joint origin so visual/collision
-  origins are (0 0 0) throughout.
+  All body_* STL meshes share the same body_link joint origin (body_shell
+  centroid) so all visual origins within body_link are (0 0 0).
+  Each wheel link has two visuals: rim (dark grey) and tire (black rubber).
+  The tire and rim STLs share the same axle-midpoint reference origin.
 -->
 <robot name="otto_starter" xmlns:xacro="http://www.ros.org/wiki/xacro">
@@ -15,5 +17,5 @@
   <!-- ══════════════════════════════════════════════════════════════════ -->
   <xacro:property name="wheel_radius"   value="0.0245"/>   <!-- m -->
-  <xacro:property name="wheel_base"     value="0.0913"/>   <!-- m  (track width) -->
+  <xacro:property name="wheel_base"     value="0.0833"/>   <!-- m  (track width) -->
   <xacro:property name="wheel_width"    value="0.008"/>    <!-- m -->
   <xacro:property name="wheel_mass"     value="0.020"/>    <!-- kg -->
@@ -32,4 +34,10 @@
     <color rgba="0.15 0.15 0.15 1.0"/>
   </material>
+  <material name="otto_dark_grey">
+    <color rgba="0.25 0.25 0.25 1.0"/>
+  </material>
+  <material name="otto_black">
+    <color rgba="0.05 0.05 0.05 1.0"/>
+  </material>
   <material name="rubber_black">
     <color rgba="0.08 0.08 0.08 1.0"/>
@@ -45,5 +53,5 @@
   </material>
   <!-- ══════════════════════════════════════════════════════════════════ -->
-  <!--  Helper macro: simple box inertia                                  -->
+  <!--  Helper macros                                                     -->
   <!-- ══════════════════════════════════════════════════════════════════ -->
   <xacro:macro name="box_inertia" params="m x y z">
@@ -79,16 +87,61 @@
   </link>
   <!-- ══════════════════════════════════════════════════════════════════ -->
-  <!--  Body shell                                                        -->
-  <!--  joint xyz from export_meshes.py:                                 -->
-  <!--    body: joint xyz="0.0231 0.0000 0.0220"                         -->
+  <!--  Body shell — multiple visuals for different colours               -->
+  <!--                                                                    -->
+  <!--  body_link joint xyz = body_shell centroid (from export script)    -->
+  <!--    body_shell:  joint xyz="0.0230 0.0000 0.0242"                  -->
+  <!--                                                                    -->
+  <!--  All sub-meshes share the same reference origin as body_shell so  -->
+  <!--  all visual origins are (0 0 0).                                   -->
   <!-- ══════════════════════════════════════════════════════════════════ -->
   <link name="body_link">
-    <visual>
-      <origin xyz="0 0 0" rpy="0 0 0"/>
-      <geometry>
-        <mesh filename="package://otto_description/meshes/body.stl"/>
+    <!-- Middle: main cylindrical shell — dark grey -->
+    <visual>
+      <origin xyz="0 0 0" rpy="0 0 0"/>
+      <geometry>
+        <mesh filename="package://otto_description/meshes/body_shell.stl"/>
+      </geometry>
+      <material name="otto_dark_grey"/>
+    </visual>
+    <!-- Middle: rear battery clips — dark grey -->
+    <visual>
+      <origin xyz="0 0 0" rpy="0 0 0"/>
+      <geometry>
+        <mesh filename="package://otto_description/meshes/body_clips.stl"/>
+      </geometry>
+      <material name="otto_dark_grey"/>
+    </visual>
+    <!-- Top: dome and cap sections — white -->
+    <visual>
+      <origin xyz="0 0 0" rpy="0 0 0"/>
+      <geometry>
+        <mesh filename="package://otto_description/meshes/body_top.stl"/>
       </geometry>
       <material name="otto_white"/>
     </visual>
+    <!-- Top: logo line engravings — black -->
+    <visual>
+      <origin xyz="0 0 0" rpy="0 0 0"/>
+      <geometry>
+        <mesh filename="package://otto_description/meshes/body_top_lines.stl"/>
+      </geometry>
+      <material name="otto_black"/>
+    </visual>
+    <!-- Unnamed COMPOUND: bottom shell — black -->
+    <visual>
+      <origin xyz="0 0 0" rpy="0 0 0"/>
+      <geometry>
+        <mesh filename="package://otto_description/meshes/body_bottom.stl"/>
+      </geometry>
+      <material name="otto_black"/>
+    </visual>
+    <!-- Unnamed COMPOUND: front face panel — dark grey -->
+    <visual>
+      <origin xyz="0 0 0" rpy="0 0 0"/>
+      <geometry>
+        <mesh filename="package://otto_description/meshes/body_face.stl"/>
+      </geometry>
+      <material name="otto_dark_grey"/>
+    </visual>
     <collision>
       <origin xyz="0 0 0" rpy="0 0 0"/>
@@ -102,18 +155,28 @@
     <parent link="base_link"/>
     <child  link="body_link"/>
-    <origin xyz="0.0265 -0.0000 0.0220" rpy="0 0 0"/>
-  </joint>
-  <!-- ══════════════════════════════════════════════════════════════════ -->
-  <!--  Wheels                                                            -->
-  <!--  joint xyz from export_meshes.py:                                 -->
-  <!--    wheel_left:  joint xyz="-0.0000 0.0416 0.0000"                 -->
-  <!--    wheel_right: joint xyz="-0.0000 -0.0416 0.0000"                -->
+    <origin xyz="0.0230 0.0000 0.0242" rpy="0 0 0"/>
+  </joint>
+  <!-- ══════════════════════════════════════════════════════════════════ -->
+  <!--  Wheels — two visuals per wheel (rim: dark grey, tyre: black)     -->
+  <!--                                                                    -->
   <!--  Meshes centred at axle midpoint — rotate around Y correctly.     -->
+  <!--  joint xyz from export_meshes.py (det=+1 transform):              -->
+  <!--    wheel_left:  joint xyz="0.0000  0.0416 0.0000"                -->
+  <!--    wheel_right: joint xyz="0.0000 -0.0416 0.0000"                -->
   <!-- ══════════════════════════════════════════════════════════════════ -->
   <link name="left_wheel_link">
-    <visual>
-      <origin xyz="0 0 0" rpy="0 0 0"/>
-      <geometry>
-        <mesh filename="package://otto_description/meshes/wheel_left.stl"/>
+    <!-- Hub + outer rim — dark grey -->
+    <visual>
+      <origin xyz="0 0 0" rpy="0 0 0"/>
+      <geometry>
+        <mesh filename="package://otto_description/meshes/wheel_left_rim.stl"/>
+      </geometry>
+      <material name="otto_dark_grey"/>
+    </visual>
+    <!-- Rubber tyre — near-black -->
+    <visual>
+      <origin xyz="0 0 0" rpy="0 0 0"/>
+      <geometry>
+        <mesh filename="package://otto_description/meshes/wheel_left_tire.stl"/>
       </geometry>
       <material name="rubber_black"/>
@@ -134,8 +197,17 @@
   </joint>
   <link name="right_wheel_link">
-    <visual>
-      <origin xyz="0 0 0" rpy="0 0 0"/>
-      <geometry>
-        <mesh filename="package://otto_description/meshes/wheel_right.stl"/>
+    <!-- Hub + outer rim — dark grey -->
+    <visual>
+      <origin xyz="0 0 0" rpy="0 0 0"/>
+      <geometry>
+        <mesh filename="package://otto_description/meshes/wheel_right_rim.stl"/>
+      </geometry>
+      <material name="otto_dark_grey"/>
+    </visual>
+    <!-- Rubber tyre — near-black -->
+    <visual>
+      <origin xyz="0 0 0" rpy="0 0 0"/>
+      <geometry>
+        <mesh filename="package://otto_description/meshes/wheel_right_tire.stl"/>
       </geometry>
       <material name="rubber_black"/>
@@ -181,5 +253,4 @@
   <!-- ══════════════════════════════════════════════════════════════════ -->
   <!--  LED Ring                                                          -->
-  <!--  joint xyz from export_meshes.py output                           -->
   <!-- ══════════════════════════════════════════════════════════════════ -->
   <link name="led_ring_link">
@@ -202,5 +273,5 @@
     <parent link="base_link"/>
     <child  link="led_ring_link"/>
-    <origin xyz="0.0231 0.0001 0.0516" rpy="0 0 0"/>
+    <origin xyz="0.0231 -0.0001 0.0516" rpy="0 0 0"/>
   </joint>
   <!-- ── Individual LED frames (positions relative to base_link) ──────
@@ -215,4 +286,5 @@
     </joint>
   </xacro:macro>
+  <!-- 13 LED pads extracted from 'LED Ring' CAF group, sorted by angle -->
   <xacro:led_frame n="0"  x="0.0049" y="-0.0104" z="0.0532"/>
   <xacro:led_frame n="1"  x="0.0126" y="-0.0181" z="0.0532"/>
@@ -220,14 +292,12 @@
   <xacro:led_frame n="3"  x="0.0336" y="-0.0181" z="0.0532"/>
   <xacro:led_frame n="4"  x="0.0412" y="-0.0104" z="0.0532"/>
-  <xacro:led_frame n="5"  x="0.0536" y="-0.0130" z="0.0310"/>
-  <xacro:led_frame n="6"  x="0.0441" y=" 0.0001" z="0.0532"/>
-  <xacro:led_frame n="7"  x="0.0231" y=" 0.0001" z="0.0532"/>
-  <xacro:led_frame n="8"  x="0.0021" y=" 0.0001" z="0.0532"/>
-  <xacro:led_frame n="9"  x="0.0536" y=" 0.0130" z="0.0310"/>
-  <xacro:led_frame n="10" x="0.0412" y=" 0.0106" z="0.0532"/>
-  <xacro:led_frame n="11" x="0.0336" y=" 0.0183" z="0.0532"/>
-  <xacro:led_frame n="12" x="0.0231" y=" 0.0211" z="0.0532"/>
-  <xacro:led_frame n="13" x="0.0126" y=" 0.0183" z="0.0532"/>
-  <xacro:led_frame n="14" x="0.0049" y=" 0.0106" z="0.0532"/>
+  <xacro:led_frame n="5"  x="0.0441" y=" 0.0001" z="0.0532"/>
+  <xacro:led_frame n="6"  x="0.0231" y=" 0.0001" z="0.0532"/>
+  <xacro:led_frame n="7"  x="0.0021" y=" 0.0001" z="0.0532"/>
+  <xacro:led_frame n="8"  x="0.0412" y=" 0.0106" z="0.0532"/>
+  <xacro:led_frame n="9"  x="0.0336" y=" 0.0183" z="0.0532"/>
+  <xacro:led_frame n="10" x="0.0231" y=" 0.0211" z="0.0532"/>
+  <xacro:led_frame n="11" x="0.0126" y=" 0.0183" z="0.0532"/>
+  <xacro:led_frame n="12" x="0.0049" y=" 0.0106" z="0.0532"/>
   <!-- ══════════════════════════════════════════════════════════════════ -->
   <!--  Ultrasonic sensor                                                 -->
@@ -252,5 +322,5 @@
     <parent link="base_link"/>
     <child  link="ultrasonic_link"/>
-    <origin xyz="0.0509 0.0000 0.0200" rpy="0 0 0"/>
+    <origin xyz="0.0520 0.0000 0.0260" rpy="0 0 0"/>
   </joint>
   <!-- Sensor ray origin — midpoint between transducers, pointing forward -->
@@ -277,5 +347,5 @@
     <parent link="base_link"/>
     <child  link="line_sensor_left_link"/>
-    <origin xyz="0.0347 0.0130 -0.0065" rpy="0 0 0"/>
+    <origin xyz="0.0347 0.0130 -0.0064" rpy="0 0 0"/>
   </joint>
   <link name="line_sensor_right_link">
@@ -292,5 +362,5 @@
     <parent link="base_link"/>
     <child  link="line_sensor_right_link"/>
-    <origin xyz="0.0347 -0.0130 -0.0065" rpy="0 0 0"/>
+    <origin xyz="0.0347 -0.0130 -0.0064" rpy="0 0 0"/>
   </joint>
   <!-- ══════════════════════════════════════════════════════════════════ -->

Commit message: Fix body top dome colour: white → black
The top dome (body_top.stl) should be black to match the physical robot,
not white as previously set.

Co-Authored-By: Claude Sonnet 4.6 <noreply@anthropic.com>

File: ros2_ws/src/otto_description/urdf/otto_starter.urdf.xacro (robot description, xacro)
@@ -112,5 +112,5 @@
       <material name="otto_dark_grey"/>
     </visual>
-    <!-- Top: dome and cap sections — white -->
+    <!-- Top: dome and cap sections — black -->
     <visual>
       <origin xyz="0 0 0" rpy="0 0 0"/>
@@ -118,5 +118,5 @@
         <mesh filename="package://otto_description/meshes/body_top.stl"/>
       </geometry>
-      <material name="otto_white"/>
+      <material name="otto_black"/>
     </visual>
     <!-- Top: logo line engravings — black -->

Commit message: Fix URDF colors: use inline rgba per visual to bypass RViz2 material name issue
RViz2 can fail to apply globally-defined named materials to multi-visual
links. Switch every visual to an inline unique material with explicit rgba
so colors are guaranteed to render: grey (0.50) for middle/rim/face,
black (0.03) for top/bottom/logo, dark rubber (0.05) for tyres.

Co-Authored-By: Claude Sonnet 4.6 <noreply@anthropic.com>

File: ros2_ws/src/otto_description/urdf/otto_starter.urdf.xacro (robot description, xacro)
@@ -96,5 +96,5 @@
   <!-- ══════════════════════════════════════════════════════════════════ -->
   <link name="body_link">
-    <!-- Middle: main cylindrical shell — dark grey -->
+    <!-- Middle: main cylindrical shell — grey -->
     <visual>
       <origin xyz="0 0 0" rpy="0 0 0"/>
@@ -102,7 +102,7 @@
         <mesh filename="package://otto_description/meshes/body_shell.stl"/>
       </geometry>
-      <material name="otto_dark_grey"/>
-    </visual>
-    <!-- Middle: rear battery clips — dark grey -->
+      <material name="body_shell_mat"><color rgba="0.50 0.50 0.50 1.0"/></material>
+    </visual>
+    <!-- Middle: rear battery clips — grey -->
     <visual>
       <origin xyz="0 0 0" rpy="0 0 0"/>
@@ -110,5 +110,5 @@
         <mesh filename="package://otto_description/meshes/body_clips.stl"/>
       </geometry>
-      <material name="otto_dark_grey"/>
+      <material name="body_clips_mat"><color rgba="0.50 0.50 0.50 1.0"/></material>
     </visual>
     <!-- Top: dome and cap sections — black -->
@@ -118,5 +118,5 @@
         <mesh filename="package://otto_description/meshes/body_top.stl"/>
       </geometry>
-      <material name="otto_black"/>
+      <material name="body_top_mat"><color rgba="0.03 0.03 0.03 1.0"/></material>
     </visual>
     <!-- Top: logo line engravings — black -->
@@ -126,7 +126,7 @@
         <mesh filename="package://otto_description/meshes/body_top_lines.stl"/>
       </geometry>
-      <material name="otto_black"/>
-    </visual>
-    <!-- Unnamed COMPOUND: bottom shell — black -->
+      <material name="body_top_lines_mat"><color rgba="0.03 0.03 0.03 1.0"/></material>
+    </visual>
+    <!-- Bottom shell — black -->
     <visual>
       <origin xyz="0 0 0" rpy="0 0 0"/>
@@ -134,7 +134,7 @@
         <mesh filename="package://otto_description/meshes/body_bottom.stl"/>
       </geometry>
-      <material name="otto_black"/>
-    </visual>
-    <!-- Unnamed COMPOUND: front face panel — dark grey -->
+      <material name="body_bottom_mat"><color rgba="0.03 0.03 0.03 1.0"/></material>
+    </visual>
+    <!-- Front face panel — grey -->
     <visual>
       <origin xyz="0 0 0" rpy="0 0 0"/>
@@ -142,5 +142,5 @@
         <mesh filename="package://otto_description/meshes/body_face.stl"/>
       </geometry>
-      <material name="otto_dark_grey"/>
+      <material name="body_face_mat"><color rgba="0.50 0.50 0.50 1.0"/></material>
     </visual>
     <collision>
@@ -166,5 +166,5 @@
   <!-- ══════════════════════════════════════════════════════════════════ -->
   <link name="left_wheel_link">
-    <!-- Hub + outer rim — dark grey -->
+    <!-- Hub + outer rim — grey -->
     <visual>
       <origin xyz="0 0 0" rpy="0 0 0"/>
@@ -172,7 +172,7 @@
         <mesh filename="package://otto_description/meshes/wheel_left_rim.stl"/>
       </geometry>
-      <material name="otto_dark_grey"/>
-    </visual>
-    <!-- Rubber tyre — near-black -->
+      <material name="left_rim_mat"><color rgba="0.50 0.50 0.50 1.0"/></material>
+    </visual>
+    <!-- Rubber tyre — black -->
     <visual>
       <origin xyz="0 0 0" rpy="0 0 0"/>
@@ -180,5 +180,5 @@
         <mesh filename="package://otto_description/meshes/wheel_left_tire.stl"/>
       </geometry>
-      <material name="rubber_black"/>
+      <material name="left_tire_mat"><color rgba="0.05 0.05 0.05 1.0"/></material>
     </visual>
     <collision>
@@ -197,5 +197,5 @@
   </joint>
   <link name="right_wheel_link">
-    <!-- Hub + outer rim — dark grey -->
+    <!-- Hub + outer rim — grey -->
     <visual>
       <origin xyz="0 0 0" rpy="0 0 0"/>
@@ -203,7 +203,7 @@
         <mesh filename="package://otto_description/meshes/wheel_right_rim.stl"/>
       </geometry>
-      <material name="otto_dark_grey"/>
-    </visual>
-    <!-- Rubber tyre — near-black -->
+      <material name="right_rim_mat"><color rgba="0.50 0.50 0.50 1.0"/></material>
+    </visual>
+    <!-- Rubber tyre — black -->
     <visual>
       <origin xyz="0 0 0" rpy="0 0 0"/>
@@ -211,5 +211,5 @@
         <mesh filename="package://otto_description/meshes/wheel_right_tire.stl"/>
       </geometry>
-      <material name="rubber_black"/>
+      <material name="right_tire_mat"><color rgba="0.05 0.05 0.05 1.0"/></material>
     </visual>
     <collision>
@@ -236,5 +236,5 @@
         <mesh filename="package://otto_description/meshes/caster.stl"/>
       </geometry>
-      <material name="otto_dark"/>
+      <material name="caster_mat"><color rgba="0.10 0.10 0.10 1.0"/></material>
     </visual>
     <collision>
