Commit message: Fix colours: split multi-visual links into one link per visual
RViz2 bug: when a link has multiple <visual> elements it applies the
first material to all of them. Fix by giving each body sub-part and
each wheel component its own dedicated link (one visual each).
Body sub-parts are all fixed children of base_link at the same origin;
rim links are fixed children of their wheel link so they rotate together.

Co-Authored-By: Claude Sonnet 4.6 <noreply@anthropic.com>

File: ros2_ws/src/otto_description/urdf/otto_starter.urdf.xacro (robot description, xacro)
@@ -95,64 +95,75 @@
   <!--  all visual origins are (0 0 0).                                   -->
   <!-- ══════════════════════════════════════════════════════════════════ -->
+  <!-- Each body sub-part is a separate link (one visual per link) because
+       RViz2 applies the first material to ALL visuals in the same link.   -->
   <link name="body_link">
-    <!-- Middle: main cylindrical shell — grey -->
-    <visual>
-      <origin xyz="0 0 0" rpy="0 0 0"/>
-      <geometry>
-        <mesh filename="package://otto_description/meshes/body_shell.stl"/>
-      </geometry>
+    <visual>
+      <origin xyz="0 0 0" rpy="0 0 0"/>
+      <geometry><mesh filename="package://otto_description/meshes/body_shell.stl"/></geometry>
       <material name="body_shell_mat"><color rgba="0.50 0.50 0.50 1.0"/></material>
     </visual>
-    <!-- Middle: rear battery clips — grey -->
-    <visual>
-      <origin xyz="0 0 0" rpy="0 0 0"/>
-      <geometry>
-        <mesh filename="package://otto_description/meshes/body_clips.stl"/>
-      </geometry>
+    <collision>
+      <origin xyz="0 0 0" rpy="0 0 0"/>
+      <geometry><box size="0.072 0.072 0.072"/></geometry>
+    </collision>
+    <xacro:box_inertia m="${body_mass}" x="0.072" y="0.072" z="0.072"/>
+  </link>
+  <joint name="body_joint" type="fixed">
+    <parent link="base_link"/><child link="body_link"/>
+    <origin xyz="0.0230 0.0000 0.0242" rpy="0 0 0"/>
+  </joint>
+  <link name="body_clips_link">
+    <visual>
+      <origin xyz="0 0 0" rpy="0 0 0"/>
+      <geometry><mesh filename="package://otto_description/meshes/body_clips.stl"/></geometry>
       <material name="body_clips_mat"><color rgba="0.50 0.50 0.50 1.0"/></material>
     </visual>
-    <!-- Top: dome and cap sections — black -->
-    <visual>
-      <origin xyz="0 0 0" rpy="0 0 0"/>
-      <geometry>
-        <mesh filename="package://otto_description/meshes/body_top.stl"/>
-      </geometry>
+  </link>
+  <joint name="body_clips_joint" type="fixed">
+    <parent link="base_link"/><child link="body_clips_link"/>
+    <origin xyz="0.0230 0.0000 0.0242" rpy="0 0 0"/>
+  </joint>
+  <link name="body_top_link">
+    <visual>
+      <origin xyz="0 0 0" rpy="0 0 0"/>
+      <geometry><mesh filename="package://otto_description/meshes/body_top.stl"/></geometry>
       <material name="body_top_mat"><color rgba="0.03 0.03 0.03 1.0"/></material>
     </visual>
-    <!-- Top: logo line engravings — black -->
-    <visual>
-      <origin xyz="0 0 0" rpy="0 0 0"/>
-      <geometry>
-        <mesh filename="package://otto_description/meshes/body_top_lines.stl"/>
-      </geometry>
+  </link>
+  <joint name="body_top_joint" type="fixed">
+    <parent link="base_link"/><child link="body_top_link"/>
+    <origin xyz="0.0230 0.0000 0.0242" rpy="0 0 0"/>
+  </joint>
+  <link name="body_top_lines_link">
+    <visual>
+      <origin xyz="0 0 0" rpy="0 0 0"/>
+      <geometry><mesh filename="package://otto_description/meshes/body_top_lines.stl"/></geometry>
       <material name="body_top_lines_mat"><color rgba="0.03 0.03 0.03 1.0"/></material>
     </visual>
-    <!-- Bottom shell — black -->
-    <visual>
-      <origin xyz="0 0 0" rpy="0 0 0"/>
-      <geometry>
-        <mesh filename="package://otto_description/meshes/body_bottom.stl"/>
-      </geometry>
+  </link>
+  <joint name="body_top_lines_joint" type="fixed">
+    <parent link="base_link"/><child link="body_top_lines_link"/>
+    <origin xyz="0.0230 0.0000 0.0242" rpy="0 0 0"/>
+  </joint>
+  <link name="body_bottom_link">
+    <visual>
+      <origin xyz="0 0 0" rpy="0 0 0"/>
+      <geometry><mesh filename="package://otto_description/meshes/body_bottom.stl"/></geometry>
       <material name="body_bottom_mat"><color rgba="0.03 0.03 0.03 1.0"/></material>
     </visual>
-    <!-- Front face panel — grey -->
-    <visual>
-      <origin xyz="0 0 0" rpy="0 0 0"/>
-      <geometry>
-        <mesh filename="package://otto_description/meshes/body_face.stl"/>
-      </geometry>
+  </link>
+  <joint name="body_bottom_joint" type="fixed">
+    <parent link="base_link"/><child link="body_bottom_link"/>
+    <origin xyz="0.0230 0.0000 0.0242" rpy="0 0 0"/>
+  </joint>
+  <link name="body_face_link">
+    <visual>
+      <origin xyz="0 0 0" rpy="0 0 0"/>
+      <geometry><mesh filename="package://otto_description/meshes/body_face.stl"/></geometry>
       <material name="body_face_mat"><color rgba="0.50 0.50 0.50 1.0"/></material>
     </visual>
-    <collision>
-      <origin xyz="0 0 0" rpy="0 0 0"/>
-      <geometry>
-        <box size="0.072 0.072 0.072"/>
-      </geometry>
-    </collision>
-    <xacro:box_inertia m="${body_mass}" x="0.072" y="0.072" z="0.072"/>
-  </link>
-  <joint name="body_joint" type="fixed">
-    <parent link="base_link"/>
-    <child  link="body_link"/>
+  </link>
+  <joint name="body_face_joint" type="fixed">
+    <parent link="base_link"/><child link="body_face_link"/>
     <origin xyz="0.0230 0.0000 0.0242" rpy="0 0 0"/>
   </joint>
@@ -166,59 +177,54 @@
   <!-- ══════════════════════════════════════════════════════════════════ -->
   <link name="left_wheel_link">
-    <!-- Hub + outer rim — grey -->
-    <visual>
-      <origin xyz="0 0 0" rpy="0 0 0"/>
-      <geometry>
-        <mesh filename="package://otto_description/meshes/wheel_left_rim.stl"/>
-      </geometry>
-      <material name="left_rim_mat"><color rgba="0.50 0.50 0.50 1.0"/></material>
-    </visual>
-    <!-- Rubber tyre — black -->
-    <visual>
-      <origin xyz="0 0 0" rpy="0 0 0"/>
-      <geometry>
-        <mesh filename="package://otto_description/meshes/wheel_left_tire.stl"/>
-      </geometry>
+    <visual>
+      <origin xyz="0 0 0" rpy="0 0 0"/>
+      <geometry><mesh filename="package://otto_description/meshes/wheel_left_tire.stl"/></geometry>
       <material name="left_tire_mat"><color rgba="0.05 0.05 0.05 1.0"/></material>
     </visual>
     <collision>
       <origin xyz="0 0 0" rpy="${pi/2} 0 0"/>
-      <geometry>
-        <cylinder radius="${wheel_radius}" length="${wheel_width}"/>
-      </geometry>
+      <geometry><cylinder radius="${wheel_radius}" length="${wheel_width}"/></geometry>
     </collision>
     <xacro:cylinder_inertia m="${wheel_mass}" r="${wheel_radius}" h="${wheel_width}"/>
   </link>
   <joint name="left_wheel_joint" type="continuous">
-    <parent link="base_link"/>
-    <child  link="left_wheel_link"/>
+    <parent link="base_link"/><child link="left_wheel_link"/>
     <origin xyz="-0.0000 0.0416 0.0000" rpy="0 0 0"/>
     <axis xyz="0 1 0"/>
   </joint>
+  <link name="left_rim_link">
+    <visual>
+      <origin xyz="0 0 0" rpy="0 0 0"/>
+      <geometry><mesh filename="package://otto_description/meshes/wheel_left_rim.stl"/></geometry>
+      <material name="left_rim_mat"><color rgba="0.50 0.50 0.50 1.0"/></material>
+    </visual>
+  </link>
+  <joint name="left_rim_joint" type="fixed">
+    <parent link="left_wheel_link"/><child link="left_rim_link"/>
+    <origin xyz="0 0 0" rpy="0 0 0"/>
+  </joint>
   <link name="right_wheel_link">
-    <!-- Hub + outer rim — grey -->
-    <visual>
-      <origin xyz="0 0 0" rpy="0 0 0"/>
-      <geometry>
-        <mesh filename="package://otto_description/meshes/wheel_right_rim.stl"/>
-      </geometry>
+    <visual>
+      <origin xyz="0 0 0" rpy="0 0 0"/>
+      <geometry><mesh filename="package://otto_description/meshes/wheel_right_tire.stl"/></geometry>
+      <material name="right_tire_mat"><color rgba="0.05 0.05 0.05 1.0"/></material>
+    </visual>
+    <collision>
+      <origin xyz="0 0 0" rpy="${pi/2} 0 0"/>
+      <geometry><cylinder radius="${wheel_radius}" length="${wheel_width}"/></geometry>
+    </collision>
+    <xacro:cylinder_inertia m="${wheel_mass}" r="${wheel_radius}" h="${wheel_width}"/>
+  </link>
+  <link name="right_rim_link">
+    <visual>
+      <origin xyz="0 0 0" rpy="0 0 0"/>
+      <geometry><mesh filename="package://otto_description/meshes/wheel_right_rim.stl"/></geometry>
       <material name="right_rim_mat"><color rgba="0.50 0.50 0.50 1.0"/></material>
     </visual>
-    <!-- Rubber tyre — black -->
-    <visual>
-      <origin xyz="0 0 0" rpy="0 0 0"/>
-      <geometry>
-        <mesh filename="package://otto_description/meshes/wheel_right_tire.stl"/>
-      </geometry>
-      <material name="right_tire_mat"><color rgba="0.05 0.05 0.05 1.0"/></material>
-    </visual>
-    <collision>
-      <origin xyz="0 0 0" rpy="${pi/2} 0 0"/>
-      <geometry>
-        <cylinder radius="${wheel_radius}" length="${wheel_width}"/>
-      </geometry>
-    </collision>
-    <xacro:cylinder_inertia m="${wheel_mass}" r="${wheel_radius}" h="${wheel_width}"/>
-  </link>
+  </link>
+  <joint name="right_rim_joint" type="fixed">
+    <parent link="right_wheel_link"/><child link="right_rim_link"/>
+    <origin xyz="0 0 0" rpy="0 0 0"/>
+  </joint>
   <joint name="right_wheel_joint" type="continuous">
     <parent link="base_link"/>

Commit message: Split caster into bracket (grey) and ball (silver)
Export caster_bracket.stl and caster_ball.stl from the two Ballcaster
solids. Bracket coloured grey (0.50) to match body; ball coloured
silver (0.80 0.80 0.85) for metallic appearance.

Co-Authored-By: Claude Sonnet 4.6 <noreply@anthropic.com>

File: ros2_ws/src/otto_description/urdf/otto_starter.urdf.xacro (robot description, xacro)
@@ -234,26 +234,38 @@
   </joint>
   <!-- ══════════════════════════════════════════════════════════════════ -->
-  <!--  Caster (front ball caster)                                        -->
+  <!--  Caster (front ball caster) — bracket grey, ball silver           -->
   <!-- ══════════════════════════════════════════════════════════════════ -->
   <link name="caster_link">
-    <visual>
-      <origin xyz="0 0 0" rpy="0 0 0"/>
-      <geometry>
-        <mesh filename="package://otto_description/meshes/caster.stl"/>
-      </geometry>
-      <material name="caster_mat"><color rgba="0.10 0.10 0.10 1.0"/></material>
-    </visual>
-    <collision>
-      <origin xyz="0 0 0" rpy="0 0 0"/>
-      <geometry>
-        <sphere radius="0.006"/>
-      </geometry>
+    <collision>
+      <origin xyz="0 0 0" rpy="0 0 0"/>
+      <geometry><sphere radius="0.006"/></geometry>
     </collision>
     <xacro:box_inertia m="${caster_mass}" x="0.012" y="0.012" z="0.012"/>
   </link>
   <joint name="caster_joint" type="fixed">
-    <parent link="base_link"/>
-    <child  link="caster_link"/>
+    <parent link="base_link"/><child link="caster_link"/>
     <origin xyz="0.0430 0.0000 -0.0190" rpy="0 0 0"/>
+  </joint>
+  <link name="caster_bracket_link">
+    <visual>
+      <origin xyz="0 0 0" rpy="0 0 0"/>
+      <geometry><mesh filename="package://otto_description/meshes/caster_bracket.stl"/></geometry>
+      <material name="caster_bracket_mat"><color rgba="0.50 0.50 0.50 1.0"/></material>
+    </visual>
+  </link>
+  <joint name="caster_bracket_joint" type="fixed">
+    <parent link="caster_link"/><child link="caster_bracket_link"/>
+    <origin xyz="0 0 0" rpy="0 0 0"/>
+  </joint>
+  <link name="caster_ball_link">
+    <visual>
+      <origin xyz="0 0 0" rpy="0 0 0"/>
+      <geometry><mesh filename="package://otto_description/meshes/caster_ball.stl"/></geometry>
+      <material name="caster_ball_mat"><color rgba="0.80 0.80 0.85 1.0"/></material>
+    </visual>
+  </link>
+  <joint name="caster_ball_joint" type="fixed">
+    <parent link="caster_link"/><child link="caster_ball_link"/>
+    <origin xyz="0 0 0" rpy="0 0 0"/>
   </joint>
   <!-- ══════════════════════════════════════════════════════════════════ -->

Commit message: Split Top Pattern from body_top: grey 60x60x2mm disc on top cap
The 'Top' STEP group's flat 60×60×2mm pattern disc is extracted into
body_top_pattern.stl (grey 0.50) as a separate link. The remaining
top solids (dome and small centre piece) stay black in body_top.stl.
export_meshes.py updated to handle this split on future re-exports.

Co-Authored-By: Claude Sonnet 4.6 <noreply@anthropic.com>

File: ros2_ws/src/otto_description/urdf/otto_starter.urdf.xacro (robot description, xacro)
@@ -133,4 +133,15 @@
   <joint name="body_top_joint" type="fixed">
     <parent link="base_link"/><child link="body_top_link"/>
+    <origin xyz="0.0230 0.0000 0.0242" rpy="0 0 0"/>
+  </joint>
+  <link name="body_top_pattern_link">
+    <visual>
+      <origin xyz="0 0 0" rpy="0 0 0"/>
+      <geometry><mesh filename="package://otto_description/meshes/body_top_pattern.stl"/></geometry>
+      <material name="body_top_pattern_mat"><color rgba="0.50 0.50 0.50 1.0"/></material>
+    </visual>
+  </link>
+  <joint name="body_top_pattern_joint" type="fixed">
+    <parent link="base_link"/><child link="body_top_pattern_link"/>
     <origin xyz="0.0230 0.0000 0.0242" rpy="0 0 0"/>
   </joint>

Commit message: Colour body clips black — 4 small Middle solids are clips, not shell
Co-Authored-By: Claude Sonnet 4.6 <noreply@anthropic.com>

File: ros2_ws/src/otto_description/urdf/otto_starter.urdf.xacro (robot description, xacro)
@@ -117,5 +117,5 @@
       <origin xyz="0 0 0" rpy="0 0 0"/>
       <geometry><mesh filename="package://otto_description/meshes/body_clips.stl"/></geometry>
-      <material name="body_clips_mat"><color rgba="0.50 0.50 0.50 1.0"/></material>
+      <material name="body_clips_mat"><color rgba="0.03 0.03 0.03 1.0"/></material>
     </visual>
   </link>

Commit message: Split wheel into 3 parts: tyre+hub black, middle rim grey
Inner hub (dia≤43mm) → wheel_*_hub.stl black (0.05)
Middle rim (43<dia≤46mm) → wheel_*_rim.stl grey (0.50)
Outer tyre (dia>46mm) → wheel_*_tire.stl black (0.05)
export_meshes.py updated with hub threshold.

Co-Authored-By: Claude Sonnet 4.6 <noreply@anthropic.com>

File: ros2_ws/src/otto_description/urdf/otto_starter.urdf.xacro (robot description, xacro)
@@ -215,4 +215,15 @@
     <origin xyz="0 0 0" rpy="0 0 0"/>
   </joint>
+  <link name="left_hub_link">
+    <visual>
+      <origin xyz="0 0 0" rpy="0 0 0"/>
+      <geometry><mesh filename="package://otto_description/meshes/wheel_left_hub.stl"/></geometry>
+      <material name="left_hub_mat"><color rgba="0.05 0.05 0.05 1.0"/></material>
+    </visual>
+  </link>
+  <joint name="left_hub_joint" type="fixed">
+    <parent link="left_wheel_link"/><child link="left_hub_link"/>
+    <origin xyz="0 0 0" rpy="0 0 0"/>
+  </joint>
   <link name="right_wheel_link">
     <visual>
@@ -236,4 +247,15 @@
   <joint name="right_rim_joint" type="fixed">
     <parent link="right_wheel_link"/><child link="right_rim_link"/>
+    <origin xyz="0 0 0" rpy="0 0 0"/>
+  </joint>
+  <link name="right_hub_link">
+    <visual>
+      <origin xyz="0 0 0" rpy="0 0 0"/>
+      <geometry><mesh filename="package://otto_description/meshes/wheel_right_hub.stl"/></geometry>
+      <material name="right_hub_mat"><color rgba="0.05 0.05 0.05 1.0"/></material>
+    </visual>
+  </link>
+  <joint name="right_hub_joint" type="fixed">
+    <parent link="right_wheel_link"/><child link="right_hub_link"/>
     <origin xyz="0 0 0" rpy="0 0 0"/>
   </joint>

Commit message: Colour LED ring: PCB blue, pads white; export led_pads.stl
- led_ring_link (PCB board): changed from pcb_green to blue (0.05 0.20 0.80)
- led_pads_link: new link with led_pads.stl in white (0.95 0.95 0.95)
- export_meshes.py: export led_pads.stl at coarse tessellation (tol=0.5mm)
  to keep file size manageable (2.5MB vs 142MB at fine tol)

Co-Authored-By: Claude Sonnet 4.6 <noreply@anthropic.com>

File: ros2_ws/src/otto_description/urdf/otto_starter.urdf.xacro (robot description, xacro)
@@ -311,5 +311,5 @@
         <mesh filename="package://otto_description/meshes/led_ring.stl"/>
       </geometry>
-      <material name="pcb_green"/>
+      <material name="led_ring_pcb_mat"><color rgba="0.05 0.20 0.80 1.0"/></material>
     </visual>
     <collision>
@@ -324,4 +324,18 @@
     <parent link="base_link"/>
     <child  link="led_ring_link"/>
+    <origin xyz="0.0231 -0.0001 0.0516" rpy="0 0 0"/>
+  </joint>
+  <link name="led_pads_link">
+    <visual>
+      <origin xyz="0 0 0" rpy="0 0 0"/>
+      <geometry>
+        <mesh filename="package://otto_description/meshes/led_pads.stl"/>
+      </geometry>
+      <material name="led_pads_mat"><color rgba="0.95 0.95 0.95 1.0"/></material>
+    </visual>
+  </link>
+  <joint name="led_pads_joint" type="fixed">
+    <parent link="base_link"/>
+    <child  link="led_pads_link"/>
     <origin xyz="0.0231 -0.0001 0.0516" rpy="0 0 0"/>
   </joint>

Commit message: Split ultrasonic sensor into 3 coloured parts
- ultrasonic_board.stl: PCB → blue (0.05 0.20 0.80)
- ultrasonic_plug.stl: rear connector → white (0.95 0.95 0.95)
- ultrasonic_metal.stl: header pins → silver (0.75 0.75 0.78), coarse tol
- Remove old single-mesh ultrasonic.stl reference from URDF
- export_meshes.py: classify by geometry (board xlen>40, plug 8<xlen, rest=pins)

Co-Authored-By: Claude Sonnet 4.6 <noreply@anthropic.com>

File: ros2_ws/src/otto_description/urdf/otto_starter.urdf.xacro (robot description, xacro)
@@ -367,25 +367,44 @@
   <!-- ══════════════════════════════════════════════════════════════════ -->
   <!--  Ultrasonic sensor                                                 -->
+  <!--  joint xyz="0.0541 -0.0000 0.0260" (board centroid, from export)  -->
+  <!--  board: blue PCB  |  plug: white connector  |  metal: silver pins -->
   <!-- ══════════════════════════════════════════════════════════════════ -->
   <link name="ultrasonic_link">
     <visual>
       <origin xyz="0 0 0" rpy="0 0 0"/>
-      <geometry>
-        <mesh filename="package://otto_description/meshes/ultrasonic.stl"/>
-      </geometry>
-      <material name="sensor_green"/>
-    </visual>
-    <collision>
-      <origin xyz="0 0 0" rpy="0 0 0"/>
-      <geometry>
-        <box size="0.010 0.005 0.006"/>
-      </geometry>
-    </collision>
-    <xacro:box_inertia m="0.002" x="0.010" y="0.005" z="0.006"/>
+      <geometry><mesh filename="package://otto_description/meshes/ultrasonic_board.stl"/></geometry>
+      <material name="us_board_mat"><color rgba="0.05 0.20 0.80 1.0"/></material>
+    </visual>
+    <collision>
+      <origin xyz="0 0 0" rpy="0 0 0"/>
+      <geometry><box size="0.046 0.002 0.021"/></geometry>
+    </collision>
+    <xacro:box_inertia m="0.002" x="0.046" y="0.002" z="0.021"/>
   </link>
   <joint name="ultrasonic_joint" type="fixed">
-    <parent link="base_link"/>
-    <child  link="ultrasonic_link"/>
-    <origin xyz="0.0520 0.0000 0.0260" rpy="0 0 0"/>
+    <parent link="base_link"/><child link="ultrasonic_link"/>
+    <origin xyz="0.0541 0.0000 0.0260" rpy="0 0 0"/>
+  </joint>
+  <link name="ultrasonic_plug_link">
+    <visual>
+      <origin xyz="0 0 0" rpy="0 0 0"/>
+      <geometry><mesh filename="package://otto_description/meshes/ultrasonic_plug.stl"/></geometry>
+      <material name="us_plug_mat"><color rgba="0.95 0.95 0.95 1.0"/></material>
+    </visual>
+  </link>
+  <joint name="ultrasonic_plug_joint" type="fixed">
+    <parent link="base_link"/><child link="ultrasonic_plug_link"/>
+    <origin xyz="0.0541 0.0000 0.0260" rpy="0 0 0"/>
+  </joint>
+  <link name="ultrasonic_metal_link">
+    <visual>
+      <origin xyz="0 0 0" rpy="0 0 0"/>
+      <geometry><mesh filename="package://otto_description/meshes/ultrasonic_metal.stl"/></geometry>
+      <material name="us_metal_mat"><color rgba="0.75 0.75 0.78 1.0"/></material>
+    </visual>
+  </link>
+  <joint name="ultrasonic_metal_joint" type="fixed">
+    <parent link="base_link"/><child link="ultrasonic_metal_link"/>
+    <origin xyz="0.0541 0.0000 0.0260" rpy="0 0 0"/>
   </joint>
   <!-- Sensor ray origin — midpoint between transducers, pointing forward -->

Commit message: Add ultrasonic transducer cans (open shells) as metallic silver
The two transducer can faces (shell_3, shell_6 CAF sub-labels) are open
shells not closed solids, missed by TopExp_Explorer(TopAbs_SOLID).
Exported as ultrasonic_cans.stl and added as us_cans_mat (silver) link.

Co-Authored-By: Claude Sonnet 4.6 <noreply@anthropic.com>

File: ros2_ws/src/otto_description/urdf/otto_starter.urdf.xacro (robot description, xacro)
@@ -408,4 +408,15 @@
     <origin xyz="0.0541 0.0000 0.0260" rpy="0 0 0"/>
   </joint>
+  <link name="ultrasonic_cans_link">
+    <visual>
+      <origin xyz="0 0 0" rpy="0 0 0"/>
+      <geometry><mesh filename="package://otto_description/meshes/ultrasonic_cans.stl"/></geometry>
+      <material name="us_cans_mat"><color rgba="0.75 0.75 0.78 1.0"/></material>
+    </visual>
+  </link>
+  <joint name="ultrasonic_cans_joint" type="fixed">
+    <parent link="base_link"/><child link="ultrasonic_cans_link"/>
+    <origin xyz="0.0541 0.0000 0.0260" rpy="0 0 0"/>
+  </joint>
   <!-- Sensor ray origin — midpoint between transducers, pointing forward -->
   <link name="ultrasonic_sensor_frame"/>
