Commit message: Split line sensors into 3 coloured parts each
- board (PCB): blue (0.05 0.20 0.80)
- white: plugs on top + potentiometer → white (0.95 0.95 0.95)
- black: IR emitter/receiver assembly on bottom front → black (0.05 0.05 0.05)

Co-Authored-By: Claude Sonnet 4.6 <noreply@anthropic.com>

File: ros2_ws/src/otto_description/urdf/otto_starter.urdf.xacro (robot description, xacro)
@@ -429,33 +429,73 @@
   <!--  Line sensors                                                      -->
   <!-- ══════════════════════════════════════════════════════════════════ -->
+  <!-- ── Line sensor left: board (blue), white parts, black IR ──────── -->
   <link name="line_sensor_left_link">
     <visual>
       <origin xyz="0 0 0" rpy="0 0 0"/>
-      <geometry>
-        <mesh filename="package://otto_description/meshes/line_sensor_left.stl"/>
-      </geometry>
-      <material name="pcb_green"/>
+      <geometry><mesh filename="package://otto_description/meshes/line_sensor_left_board.stl"/></geometry>
+      <material name="ls_left_board_mat"><color rgba="0.05 0.20 0.80 1.0"/></material>
     </visual>
     <xacro:box_inertia m="0.003" x="0.014" y="0.034" z="0.002"/>
   </link>
   <joint name="line_sensor_left_joint" type="fixed">
-    <parent link="base_link"/>
-    <child  link="line_sensor_left_link"/>
-    <origin xyz="0.0347 0.0130 -0.0064" rpy="0 0 0"/>
-  </joint>
+    <parent link="base_link"/><child link="line_sensor_left_link"/>
+    <origin xyz="0.0347 0.0130 -0.0065" rpy="0 0 0"/>
+  </joint>
+  <link name="line_sensor_left_white_link">
+    <visual>
+      <origin xyz="0 0 0" rpy="0 0 0"/>
+      <geometry><mesh filename="package://otto_description/meshes/line_sensor_left_white.stl"/></geometry>
+      <material name="ls_left_white_mat"><color rgba="0.95 0.95 0.95 1.0"/></material>
+    </visual>
+  </link>
+  <joint name="line_sensor_left_white_joint" type="fixed">
+    <parent link="base_link"/><child link="line_sensor_left_white_link"/>
+    <origin xyz="0.0347 0.0130 -0.0065" rpy="0 0 0"/>
+  </joint>
+  <link name="line_sensor_left_black_link">
+    <visual>
+      <origin xyz="0 0 0" rpy="0 0 0"/>
+      <geometry><mesh filename="package://otto_description/meshes/line_sensor_left_black.stl"/></geometry>
+      <material name="ls_left_black_mat"><color rgba="0.05 0.05 0.05 1.0"/></material>
+    </visual>
+  </link>
+  <joint name="line_sensor_left_black_joint" type="fixed">
+    <parent link="base_link"/><child link="line_sensor_left_black_link"/>
+    <origin xyz="0.0347 0.0130 -0.0065" rpy="0 0 0"/>
+  </joint>
+  <!-- ── Line sensor right: board (blue), white parts, black IR ─────── -->
   <link name="line_sensor_right_link">
     <visual>
       <origin xyz="0 0 0" rpy="0 0 0"/>
-      <geometry>
-        <mesh filename="package://otto_description/meshes/line_sensor_right.stl"/>
-      </geometry>
-      <material name="pcb_green"/>
+      <geometry><mesh filename="package://otto_description/meshes/line_sensor_right_board.stl"/></geometry>
+      <material name="ls_right_board_mat"><color rgba="0.05 0.20 0.80 1.0"/></material>
     </visual>
     <xacro:box_inertia m="0.003" x="0.014" y="0.034" z="0.002"/>
   </link>
   <joint name="line_sensor_right_joint" type="fixed">
-    <parent link="base_link"/>
-    <child  link="line_sensor_right_link"/>
-    <origin xyz="0.0347 -0.0130 -0.0064" rpy="0 0 0"/>
+    <parent link="base_link"/><child link="line_sensor_right_link"/>
+    <origin xyz="0.0347 -0.0130 -0.0065" rpy="0 0 0"/>
+  </joint>
+  <link name="line_sensor_right_white_link">
+    <visual>
+      <origin xyz="0 0 0" rpy="0 0 0"/>
+      <geometry><mesh filename="package://otto_description/meshes/line_sensor_right_white.stl"/></geometry>
+      <material name="ls_right_white_mat"><color rgba="0.95 0.95 0.95 1.0"/></material>
+    </visual>
+  </link>
+  <joint name="line_sensor_right_white_joint" type="fixed">
+    <parent link="base_link"/><child link="line_sensor_right_white_link"/>
+    <origin xyz="0.0347 -0.0130 -0.0065" rpy="0 0 0"/>
+  </joint>
+  <link name="line_sensor_right_black_link">
+    <visual>
+      <origin xyz="0 0 0" rpy="0 0 0"/>
+      <geometry><mesh filename="package://otto_description/meshes/line_sensor_right_black.stl"/></geometry>
+      <material name="ls_right_black_mat"><color rgba="0.05 0.05 0.05 1.0"/></material>
+    </visual>
+  </link>
+  <joint name="line_sensor_right_black_joint" type="fixed">
+    <parent link="base_link"/><child link="line_sensor_right_black_link"/>
+    <origin xyz="0.0347 -0.0130 -0.0065" rpy="0 0 0"/>
   </joint>
   <!-- ══════════════════════════════════════════════════════════════════ -->

Commit message: Add ultrasonic LED frames and RViz visualisation
6× WS2812B NeoPixels on the ultrasonic PCB are now represented in RViz.
3 LEDs per emitter, equally spaced at r=4mm from each transducer centre
(y=±0.013m from board centre). Reference LED at robot-right (−Y) per emitter.

URDF: us_led_0..5_link fixed frames under ultrasonic_link.
Visualizer: /otto/us_led_markers MarkerArray, colour mirrors firmware
led_proximity() logic (red=near, orange=mid, green=far).

Firmware index → frame mapping TBD (calibrate physically).

Co-Authored-By: Claude Sonnet 4.6 <noreply@anthropic.com>

File: ros2_ws/src/otto_description/urdf/otto_starter.urdf.xacro (robot description, xacro)
@@ -426,4 +426,40 @@
     <origin xyz="0 0 0" rpy="0 0 0"/>
   </joint>
+  <!-- 6× WS2812B NeoPixels on ultrasonic PCB — 3 per emitter at r=4mm.
+       Numbering: 0-2 = right emitter, 3-5 = left emitter.
+       Within each group: index 0/3 = rightmost LED (−Y), then 120° CCW steps.
+       Firmware LED index → frame mapping TBD (calibrate physically). -->
+  <!-- Right emitter  centre y=−0.0130 -->
+  <link name="us_led_0_link"/>
+  <joint name="us_led_0_joint" type="fixed">
+    <parent link="ultrasonic_link"/><child link="us_led_0_link"/>
+    <origin xyz="0.0000 -0.0170  0.0000"/>
+  </joint>
+  <link name="us_led_1_link"/>
+  <joint name="us_led_1_joint" type="fixed">
+    <parent link="ultrasonic_link"/><child link="us_led_1_link"/>
+    <origin xyz="0.0000 -0.0110  0.0035"/>
+  </joint>
+  <link name="us_led_2_link"/>
+  <joint name="us_led_2_joint" type="fixed">
+    <parent link="ultrasonic_link"/><child link="us_led_2_link"/>
+    <origin xyz="0.0000 -0.0110 -0.0035"/>
+  </joint>
+  <!-- Left emitter  centre y=+0.0130 -->
+  <link name="us_led_3_link"/>
+  <joint name="us_led_3_joint" type="fixed">
+    <parent link="ultrasonic_link"/><child link="us_led_3_link"/>
+    <origin xyz="0.0000  0.0090  0.0000"/>
+  </joint>
+  <link name="us_led_4_link"/>
+  <joint name="us_led_4_joint" type="fixed">
+    <parent link="ultrasonic_link"/><child link="us_led_4_link"/>
+    <origin xyz="0.0000  0.0150  0.0035"/>
+  </joint>
+  <link name="us_led_5_link"/>
+  <joint name="us_led_5_joint" type="fixed">
+    <parent link="ultrasonic_link"/><child link="us_led_5_link"/>
+    <origin xyz="0.0000  0.0150 -0.0035"/>
+  </joint>
   <!-- ══════════════════════════════════════════════════════════════════ -->
   <!--  Line sensors                                                      -->

Commit message: Fix US LED positions: move inside cans and correct left/right
- x=0 was inside the PCB mesh; move to x=0.003 (inside can opening)
- Reference LED dy sign was inverted; flip to +Y so reference appears right

Co-Authored-By: Claude Sonnet 4.6 <noreply@anthropic.com>

File: ros2_ws/src/otto_description/urdf/otto_starter.urdf.xacro (robot description, xacro)
@@ -427,6 +427,7 @@
   </joint>
   <!-- 6× WS2812B NeoPixels on ultrasonic PCB — 3 per emitter at r=4mm.
+       x=0.003: inside the can opening, just past the PCB front face.
        Numbering: 0-2 = right emitter, 3-5 = left emitter.
-       Within each group: index 0/3 = rightmost LED (−Y), then 120° CCW steps.
+       Within each group: index 0/3 = rightmost LED (+Y), then 120° CCW steps.
        Firmware LED index → frame mapping TBD (calibrate physically). -->
   <!-- Right emitter  centre y=−0.0130 -->
@@ -434,15 +435,15 @@
   <joint name="us_led_0_joint" type="fixed">
     <parent link="ultrasonic_link"/><child link="us_led_0_link"/>
-    <origin xyz="0.0000 -0.0170  0.0000"/>
+    <origin xyz="0.0030 -0.0090  0.0000"/>
   </joint>
   <link name="us_led_1_link"/>
   <joint name="us_led_1_joint" type="fixed">
     <parent link="ultrasonic_link"/><child link="us_led_1_link"/>
-    <origin xyz="0.0000 -0.0110  0.0035"/>
+    <origin xyz="0.0030 -0.0150  0.0035"/>
   </joint>
   <link name="us_led_2_link"/>
   <joint name="us_led_2_joint" type="fixed">
     <parent link="ultrasonic_link"/><child link="us_led_2_link"/>
-    <origin xyz="0.0000 -0.0110 -0.0035"/>
+    <origin xyz="0.0030 -0.0150 -0.0035"/>
   </joint>
   <!-- Left emitter  centre y=+0.0130 -->
@@ -450,15 +451,15 @@
   <joint name="us_led_3_joint" type="fixed">
     <parent link="ultrasonic_link"/><child link="us_led_3_link"/>
-    <origin xyz="0.0000  0.0090  0.0000"/>
+    <origin xyz="0.0030  0.0170  0.0000"/>
   </joint>
   <link name="us_led_4_link"/>
   <joint name="us_led_4_joint" type="fixed">
     <parent link="ultrasonic_link"/><child link="us_led_4_link"/>
-    <origin xyz="0.0000  0.0150  0.0035"/>
+    <origin xyz="0.0030  0.0110  0.0035"/>
   </joint>
   <link name="us_led_5_link"/>
   <joint name="us_led_5_joint" type="fixed">
     <parent link="ultrasonic_link"/><child link="us_led_5_link"/>
-    <origin xyz="0.0000  0.0150 -0.0035"/>
+    <origin xyz="0.0030  0.0110 -0.0035"/>
   </joint>
   <!-- ══════════════════════════════════════════════════════════════════ -->

Commit message: Fix US LED radius to 4.5mm and add RViz display
- URDF: increase LED radius 4mm→4.5mm from each emitter centre
- RViz: add /otto/us_led_markers MarkerArray display (was missing, so no colours shown)

Co-Authored-By: Claude Sonnet 4.6 <noreply@anthropic.com>

File: ros2_ws/src/otto_description/urdf/otto_starter.urdf.xacro (robot description, xacro)
@@ -426,5 +426,5 @@
     <origin xyz="0 0 0" rpy="0 0 0"/>
   </joint>
-  <!-- 6× WS2812B NeoPixels on ultrasonic PCB — 3 per emitter at r=4mm.
+  <!-- 6× WS2812B NeoPixels on ultrasonic PCB — 3 per emitter at r=4.5mm.
        x=0.003: inside the can opening, just past the PCB front face.
        Numbering: 0-2 = right emitter, 3-5 = left emitter.
@@ -435,15 +435,15 @@
   <joint name="us_led_0_joint" type="fixed">
     <parent link="ultrasonic_link"/><child link="us_led_0_link"/>
-    <origin xyz="0.0030 -0.0090  0.0000"/>
+    <origin xyz="0.0030 -0.0085  0.0000"/>
   </joint>
   <link name="us_led_1_link"/>
   <joint name="us_led_1_joint" type="fixed">
     <parent link="ultrasonic_link"/><child link="us_led_1_link"/>
-    <origin xyz="0.0030 -0.0150  0.0035"/>
+    <origin xyz="0.0030 -0.0153  0.0039"/>
   </joint>
   <link name="us_led_2_link"/>
   <joint name="us_led_2_joint" type="fixed">
     <parent link="ultrasonic_link"/><child link="us_led_2_link"/>
-    <origin xyz="0.0030 -0.0150 -0.0035"/>
+    <origin xyz="0.0030 -0.0153 -0.0039"/>
   </joint>
   <!-- Left emitter  centre y=+0.0130 -->
@@ -451,15 +451,15 @@
   <joint name="us_led_3_joint" type="fixed">
     <parent link="ultrasonic_link"/><child link="us_led_3_link"/>
-    <origin xyz="0.0030  0.0170  0.0000"/>
+    <origin xyz="0.0030  0.0175  0.0000"/>
   </joint>
   <link name="us_led_4_link"/>
   <joint name="us_led_4_joint" type="fixed">
     <parent link="ultrasonic_link"/><child link="us_led_4_link"/>
-    <origin xyz="0.0030  0.0110  0.0035"/>
+    <origin xyz="0.0030  0.0108  0.0039"/>
   </joint>
   <link name="us_led_5_link"/>
   <joint name="us_led_5_joint" type="fixed">
     <parent link="ultrasonic_link"/><child link="us_led_5_link"/>
-    <origin xyz="0.0030  0.0110 -0.0035"/>
+    <origin xyz="0.0030  0.0108 -0.0039"/>
   </joint>
   <!-- ══════════════════════════════════════════════════════════════════ -->
